File: GateDriverPCB/GateDriver/GateDriver.sch (KiCad schematic (older format))
At the start: 25 parts

Commit message: Finished Gate Driver Schematic. Only connectors for connection to Inverter PCB need to be placed.
Parts:
- removed D?: D_Schottky_ALT, symbol Device:D_Schottky_ALT
- removed PS?: ITX4812SA, Converter_DCDC:Converter_DCDC_XP_POWER-ITXxxxxSA_THT, symbol Converter_DCDC:ITX4812SA
- added C? (x3): 0.1u, symbol Device:C
- added C? (x4): 1u, symbol Device:C_Small
- added C? (x4): 0.1u, symbol Device:C_Small
- added C? (x2): 10u, symbol Device:C_Small
- added C? (x2): Cgs, symbol Device:C
- added C? (x4): 0.01u, symbol Device:C_Small
- added C? (x2): 1000p, symbol Device:C_Small
- added C?: 0.022u, Capacitor_SMD:C_0805_2012Metric_Pad1.18x1.45mm_HandSolder, symbol Device:C
- added C? (x2): 0.47u, Capacitor_SMD:C_0805_2012Metric_Pad1.18x1.45mm_HandSolder, symbol Device:C
- added D?: RB511SM-30, Diode_SMD:D_SOD-523, symbol Device:D_Schottky_ALT
- added D? (x2): VS-30BQ015-M3, Diode_SMD:D_SMC_Handsoldering, symbol Device:D_Schottky_ALT
- added PS?: ITX4812SA, Converter_DCDC:Converter_DCDC_XP_POWER-ITXxxxxSA_THT, symbol Converter_DCDC:ITX4812SA
- added R? (x2): Ron, symbol Device:R
- added R? (x2): Roff, symbol Device:R
- D?: value D_Schottky_ALT -> RB511SM-30; footprint (none) -> Diode_SMD:D_SOD-523
- U?: value 2EDS8265 -> SN74AUP2G08; footprint (none) -> XFootprintLib:R-PDSO-G8
- U? (x3): value SN74AUP2G17 -> SN74AUP2G08; footprint XFootprintLib:DCK_R-PDSO-G6 -> XFootprintLib:R-PDSO-G8
- U? (x3): value SN74AUP2G00 -> SN74AUP2G08; footprint (none) -> XFootprintLib:R-PDSO-G8
- U? (x3): footprint (none) -> XFootprintLib:R-PDSO-G8
- U?: value TPS7B81 -> SN74AUP2G08; footprint (none) -> XFootprintLib:R-PDSO-G8
Connections:
- net +12V_ISO1: now also C?.2, C?.2, C?.2, C?.2, C?.2, C?.2, C?.2, C?.2, C?.2, C?.2, C?.2, PS?.6 (+Vout)
- net +12V_ISO2: now also C?.2
- net +3V3: now also U?.5 (VCC), U?.8 (SLDON), U?.8 (VCC), U?.8 (VCC), C?.1, C?.1, C?.1, C?.1
- net +BATT: now also C?.2, C?.2, C?.2, C?.2, C?.2, C?.2, PS?.2 (+Vin)
- net -BATT: now also C?.1, C?.1, C?.1, C?.1, C?.1, C?.1, PS?.1 (-Vin)
- net GND: now also U?.2 (GND), U?.4 (GND), U?.4 (GND), U?.5 (DISABLE), C?.2, C?.2, C?.2, C?.2
- net GND_ISO1: now also C?.1, C?.1, C?.1, C?.1, C?.1, C?.1, C?.1, C?.1, C?.1, C?.1, C?.1, C?.2, PS?.7 (-Vout)
- net GND_ISO2: now also C?.1, C?.2
- net PWM_IN_HI: now also D?.1 (K)
- net at U?.10 (OUTB): now also R?.2, R?.2
- net at U?.15 (OUTA): now also R?.2, R?.2
- net at C?.1, R?.1, U?.1 (1A): now also D?.2 (A)
- new net: D?.1 (K), R?.1 (x2)
- new net Gate_HI: C?.1, D?.2 (A), R?.1
- new net Gate_LO: C?.1, D?.2 (A), R?.1
Other:
- note added: "R_G"
- moved on the sheet: U?A, U?B, U?C

Commit message: Finished PCB layout for Gate Driver, Inverter Leg and DC Link PCB.
Parts:
- removed D?: VS-30BQ015-M3, Diode_SMD:D_SMC_Handsoldering, symbol Device:D_Schottky_ALT
- removed U?: SN74AUP2G08, XFootprintLib:R-PDSO-G8, symbol XCompLib:2EDS8265
- removed U? (x3): SN74AUP2G08, XFootprintLib:R-PDSO-G8, symbol XCompLib:SN74AUP2G17
- removed U? (x3): SN74AUP2G08, XFootprintLib:R-PDSO-G8, symbol XCompLib:SN74AUP2G00
- added D3: V3PM6-M3/I, XFootprintLib:D_SMP_DO-220AA, symbol Device:D_Schottky_ALT
- added J4: Molex KK, Connector_Molex:Molex_KK-254_AE-6410-04A_1x04_P2.54mm_Vertical, symbol Connector_Generic:Conn_01x04
- added J5, J6: SAMTEC_HMTSW, Connector_PinHeader_2.54mm:PinHeader_2x02_P2.54mm_Vertical, symbol Connector_Generic:Conn_02x02_Odd_Even
- added U2: 2EDS8265, XFootprintLib:PG-DSO-16-30, symbol XCompLib:2EDS8265
- added U3: SN74AUP2G17, XFootprintLib:DCK_R-PDSO-G6, symbol XCompLib:SN74AUP2G17
- added U5: SN74AUP2G00, XFootprintLib:R-PDSO-G8, symbol XCompLib:SN74AUP2G00
- C1, C10, C11, C12, C16, C17, C18, C19, C2, C20, C21, C22, C23, C24, C25, C26, C27, C28, C29, C3, C4, C5, C6, C7, C8, C9: renamed from C?; footprint (none) -> Capacitor_SMD:C_0805_2012Metric
- C13, C14, C15: renamed from C?; footprint Capacitor_SMD:C_0805_2012Metric_Pad1.18x1.45mm_HandSolder -> Capacitor_SMD:C_0805_2012Metric
- D1: renamed from D?; value VS-30BQ015-M3 -> V3PM6-M3/I; footprint Diode_SMD:D_SMC_Handsoldering -> XFootprintLib:D_SMP_DO-220AA
- J1, J3: renamed from J?; value Conn_01x02 -> Molex KK; footprint (none) -> Connector_Molex:Molex_KK-254_AE-6410-04A_1x04_P2.54mm_Vertical; symbol Connector_Generic:Conn_01x02 -> Connector_Generic:Conn_01x04
- J2: renamed from J?; value Conn_01x02 -> SAMTEC_HMTSW; footprint (none) -> Connector_PinHeader_2.54mm:PinHeader_2x02_P2.54mm_Vertical; symbol Connector_Generic:Conn_01x02 -> Connector_Generic:Conn_02x02_Odd_Even; Part No. (none) -> HMTSW-102-22-L-D-370
- R1, R2, R4, R5: renamed from R?; footprint (none) -> Resistor_SMD:R_1206_3216Metric
- R3, R6: renamed from R?; footprint (none) -> Resistor_SMD:R_0805_2012Metric
- U1: renamed from U?; footprint XFootprintLib:R-PDSO-G8 -> XFootprintLib:TI-VSSOP-8-PowerPAD
- gave numbers to parts that had none: 5
Connections:
- net +12V: now also J1.2 (Pin_2), J4.1 (Pin_1), J4.2 (Pin_2)
- net +12V_ISO1: now also U2.16 (VDDA); no longer C22.2, C23.2, C24.2, C25.2, C26.2, PS2.6 (+Vout)
- net +12V_ISO2: now also C22.2, C23.2, C24.2, C25.2, C26.2, PS2.6 (+Vout), U2.11 (VDDB)
- net +3V3: now also U2.3 (VDDI), U2.8 (SLDON), U3.5 (VCC), U5.8 (VCC)
- net +BATT: now also J2.2 (Pin_2)
- net -BATT: now also J2.3 (Pin_3), J2.4 (Pin_4); no longer J2.2 (Pin_2)
- net GND: now also J1.3 (Pin_3), J1.4 (Pin_4), J3.2 (Pin_2), J3.4 (Pin_4), J4.3 (Pin_3), J4.4 (Pin_4), U2.4 (GNDI), U2.5 (DISABLE), U3.2 (GND), U5.4 (GND); no longer J1.2 (Pin_2)
- net GND_ISO1: now also J5.2 (Pin_2), J5.4 (Pin_4), U2.14 (GNDA); no longer C22.1, C23.1, C24.1, C25.1, C26.1, PS2.7 (-Vout)
- net GND_ISO2: now also C22.1, C23.1, C24.1, C25.1, C26.1, PS2.7 (-Vout), J6.2 (Pin_2), J6.4 (Pin_4), U2.9 (GNDB)
- net Gate_HI: now also J5.1 (Pin_1), J5.3 (Pin_3)
- net Gate_LO: now also D3.2 (A), J6.1 (Pin_1), J6.3 (Pin_3)
- net PWM_H: now also U2.1 (INA)
- net PWM_IN_LO: now also J3.3 (Pin_3); no longer J3.2 (Pin_2)
- net PWM_L: now also U2.2 (INB)
- net at C16.1, D2.2 (A), R3.1: now also U3.3 (2A)
- net at R4.2, R5.2: now also U2.10 (OUTB)
- net at R1.2, R2.2: now also U2.15 (OUTA)
- net at U4.1 (1A): now also U3.4 (2Y), U5.1 (1A), U5.2 (1B)
- net at C18.1, D4.2 (A), R6.1: now also U3.1 (1A)
- net at U4.6 (2B): now also U3.6 (1Y), U5.5 (2A), U5.6 (2B)
- net at U4.5 (2A): now also U5.7 (1Y)
- net at U4.2 (1B): now also U5.3 (2Y)
- net at R4.1: now also D3.1 (K)
Other:
- note added: "From Interface Board / \nPrevious Gate Driver"
- note added: "Gate Driver Signals"
- note added: "To next Gate\nDriver"
- moved on the sheet: C12, C17, C18
